File: Projet_KICAD/Projet_PCBPolytech_git.kicad_pcb (KiCad board)
At the start: 2 copper layers, 35 x 20 mm, 0 parts

Commit message: start pcb design
Parts:
- added C1: 100n, Capacitor_SMD:C_0805_2012Metric, F.Cu at (125.5, 82.8)
- added C10: 100n, Capacitor_SMD:C_0805_2012Metric, F.Cu at (125.5, 97.8)
- added C11: 100n, Capacitor_SMD:C_0805_2012Metric, F.Cu at (130.0, 82.8)
- added C12: 1u, Capacitor_SMD:C_0805_2012Metric, F.Cu at (130.0, 85.8)
- added C13: 1u, Capacitor_SMD:C_0805_2012Metric, F.Cu at (130.0, 88.8)
- added C14: 100n, Capacitor_SMD:C_0805_2012Metric, F.Cu at (130.0, 91.8)
- added C15: 100n, Capacitor_SMD:C_0805_2012Metric, F.Cu at (130.0, 94.8)
- added C2: 100n, Capacitor_SMD:C_0805_2012Metric, F.Cu at (125.5, 85.8)
- added C3: 100n, Capacitor_SMD:C_0603_1608Metric, F.Cu at (159.2, 108.9)
- added C4: 100n, Capacitor_SMD:C_0603_1608Metric, F.Cu at (159.2, 111.4)
- added C5: 4.7u, Capacitor_SMD:C_0805_2012Metric, F.Cu at (125.5, 88.8)
- added C6: 100n, Capacitor_SMD:C_0603_1608Metric, F.Cu at (159.2, 113.9)
- added C7: 100n, Capacitor_SMD:C_0603_1608Metric, F.Cu at (159.2, 116.4)
- added C8: 4.7u, Capacitor_SMD:C_0805_2012Metric, F.Cu at (125.5, 91.8)
- added C9: 1u, Capacitor_SMD:C_0805_2012Metric, F.Cu at (125.5, 94.8)
- added D1: LED, LED_SMD:LED_0805_2012Metric, F.Cu at (135.4, 107.0)
- added D2: LED, LED_SMD:LED_0805_2012Metric, F.Cu at (135.4, 113.5)
- added J1: SWD, Connector_PinHeader_2.54mm:PinHeader_1x05_P2.54mm_Vertical, F.Cu at (134.5, 83.5)
- added J2: USB_B_Micro, Connector_USB:USB_Micro-AB_Molex_47590-0001, F.Cu at (151.5, 112.6)
- added J3: Conn_01x05_Socket, Connector_PinHeader_2.54mm:PinHeader_1x05_P2.54mm_Vertical, F.Cu at (139.1, 83.5)
- added Q1: BSS138, Package_TO_SOT_SMD:SOT-23, F.Cu at (156.7, 98.2)
- added Q2: BSS138, Package_TO_SOT_SMD:SOT-23, F.Cu at (156.7, 102.7)
- added R1: 10k, Resistor_SMD:R_0805_2012Metric, F.Cu at (125.5, 100.8)
- added R10: 4.7K, Resistor_SMD:R_0805_2012Metric, F.Cu at (129.9, 109.6)
- added R11: 4.7K, Resistor_SMD:R_0805_2012Metric, F.Cu at (129.9, 112.6)
- added R2: 1K, Resistor_SMD:R_0805_2012Metric, F.Cu at (125.5, 103.7)
- added R3: 10K, Resistor_SMD:R_0805_2012Metric, F.Cu at (125.5, 106.7)
- added R4: 1K, Resistor_SMD:R_0805_2012Metric, F.Cu at (125.5, 109.6)
- added R5: 10K, Resistor_SMD:R_0805_2012Metric, F.Cu at (125.5, 112.6)
- added R6: 10k, Resistor_SMD:R_0805_2012Metric, F.Cu at (125.5, 115.5)
- added R7: 10K, Resistor_SMD:R_0805_2012Metric, F.Cu at (129.9, 100.8)
- added R8: 4.7K, Resistor_SMD:R_0805_2012Metric, F.Cu at (129.9, 103.7)
- added R9: 4.7K, Resistor_SMD:R_0805_2012Metric, F.Cu at (129.9, 106.7)
- added SW1: SW_Push, Button_Switch_SMD:SW_Push_1P1T_NO_CK_KSC6xxG, F.Cu at (139.0, 99.9)
- added U1: PM004MNIATR, easyeda2kicad:SOP-8_L4.9-W3.9-P1.27-LS6.0-BL, F.Cu at (142.1, 107.9)
- added U2: STM32F446RETx, Package_QFP:LQFP-64_10x10mm_P0.5mm, F.Cu at (148.6, 88.5)
- added U3: AP2112K-3.3, Package_TO_SOT_SMD:SOT-23-5, F.Cu at (158.4, 83.7)
- added U4: USBLC6-2SC6, Package_TO_SOT_SMD:SOT-23-6_Handsoldering, F.Cu at (141.6, 114.5)
- added U5: CH340C, Package_SO:SOIC-16_3.9x9.9mm_P1.27mm, F.Cu at (150.0, 101.9)
Other:
- board size 35 x 20 mm -> 7.5 x 2 mm
- copper layers 2 -> 4

Commit message: first version of PCB, a little change of shema
Parts:
- moved U3 138.0 mm to (27.4, 40.3)
- moved C4 115.7 mm to (72.9, 34.2)
- moved C6 114.9 mm to (72.9, 38.0)
- moved C7 114.0 mm to (73.0, 41.8)
- moved U1 97.2 mm to (59.3, 56.9)
- moved C1 97.1 mm to (28.6, 77.4)
- moved C9 97.1 mm to (28.5, 90.9)
- moved C10 97.1 mm to (28.5, 94.3)
- moved R1 97.1 mm to (28.5, 97.7)
- moved C2 97.1 mm to (28.6, 80.8)
- moved R2 97.0 mm to (28.5, 101.1)
- moved R3 97.0 mm to (28.6, 104.4)
- moved R4 96.9 mm to (28.6, 107.8)
- moved R5 96.9 mm to (28.6, 111.1)
- moved R6 96.8 mm to (28.7, 114.5)
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Routing:
- net GND: track 0.00 -> 58.5 mm, vias 0 -> 34
- net +3V3: track 0.00 -> 47.6 mm, vias 0 -> 29
- net /RESET_STM_N: track 0.00 -> 16.6 mm, vias 0 -> 1
- net /JTCK-SWCLK: track 0.00 -> 16.1 mm
- net /I2C1_SCL: track 0.00 -> 12.5 mm
- net /JTMS-SWDIO: track 0.00 -> 10.2 mm
- net /I2C1_SDA: track 0.00 -> 9.80 mm
- net Net-(U2-BOOT0): track 0.00 -> 6.62 mm
- net Net-(U2-VCAP_1): track 0.00 -> 5.95 mm
- net /RTC_SDA_5V: track 0.00 -> 2.39 mm
- net /RTC_SCL_5V: track 0.00 -> 2.25 mm
Other:
- board size 7.5 x 2 mm -> 71.7 x 52.7 mm

Commit message: second version of PCB, connection
Parts:
- moved U3 159.7 mm to (174.9, 101.3)
- moved C2 157.2 mm to (184.8, 98.3), turned to 180 degrees
- moved C10 153.9 mm to (181.7, 79.9), turned to 180 degrees
- moved C9 150.3 mm to (178.7, 85.7), turned to 90 degrees
- moved C11 147.9 mm to (182.1, 85.7), turned to 90 degrees
- moved C13 145.6 mm to (179.0, 100.8)
- moved C12 138.5 mm to (171.5, 100.4), turned to -90 degrees
- moved U1 137.2 mm to (189.2, 101.0)
- moved C4 133.7 mm to (193.9, 91.2), turned to 180 degrees
- moved C6 132.1 mm to (198.2, 79.9), turned to -90 degrees
- moved C15 128.1 mm to (162.3, 96.4), turned to 180 degrees
- moved C14 126.7 mm to (161.0, 86.3)
- moved C7 118.2 mm to (186.3, 75.2)
- moved U4 106.9 mm to (166.7, 98.8), turned to 90 degrees
- moved J2 94.7 mm to (166.4, 108.2)
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Routing:
- net +5V: track 0.00 -> 19.9 mm
- net /JTCK-SWCLK: track 16.1 -> 9.07 mm
- net /USB_D+: track 0.00 -> 5.32 mm
- net /USB_D-: track 0.00 -> 5.25 mm
- net +3V3: track 47.6 -> 52.3 mm, vias 29 -> 17
- net /CH340C UD-: track 0.00 -> 3.76 mm
- net /CH340C UD+: track 0.00 -> 3.75 mm
- net GND: track 58.5 -> 61.5 mm, vias 34 -> 25
- net Net-(U2-BOOT0): track 6.62 -> 7.85 mm
- net /I2C1_SCL: track 12.5 -> 13.2 mm
- net /I2C1_SDA: track 9.80 -> 10.4 mm
