File: Projet_KICAD/Projet_PCBPolytech_git.kicad_sch (KiCad schematic)
At the start: 14 parts, among them J1 Conn_01x05_Socket, J2 USB_B_Micro, SW1 SW_Push, U1 STM32F446RETx, U2 USBLC6-2SC6

Commit message: first version of schemic , wait for complete
Parts:
- added C10, C4: 4.7u, symbol Device:C
- added C11, C9: 100n, symbol Device:C
- added C12: 1u, symbol Device:C
- added C13, C14: 1u, Package_QFP:PQFP-160_28x28mm_P0.65mm, symbol Device:C
- added C5, C6, C7, C8: 100n, Capacitor_SMD:C_0603_1608Metric, symbol Device:C
- added J3: Conn_01x05_Socket, Connector_PinHeader_2.54mm:PinHeader_1x05_P2.54mm_Vertical, symbol Connector:Conn_01x05_Socket
- added R5, R6: R, Resistor_SMD:R_0805_2012Metric, symbol Device:R
- added U3: AP2112K-3.3, Package_TO_SOT_SMD:SOT-23-5, symbol Regulator_Linear:AP2112K-3.3
Connections:
- net +3V3: now also U1.1 (VBAT), U1.13 (VDDA), U1.19 (VDD), U1.32 (VDD), U1.48 (VDD), U1.64 (VDD), C10.1, C11.1, C12.1, C14.1, C5.1, C6.1, C7.1, C8.1, C9.1, R5.1, R6.1, U3.5 (VOUT)
- net +5V: now also C13.1, U3.1 (VIN), U3.3 (EN)
- net GND: now also J2.5 (GND), U1.12 (VSSA), U1.18 (VSS), U1.31 (VSS), U1.47 (VSS), U1.63 (VSS), C10.2, C11.2, C12.2, C13.2, C14.2, C4.2, C5.2, C6.2, C7.2, C8.2, C9.2, J3.1 (Pin_1), U3.2 (GND)
- net UART4_TX: now reaches U1.14 (PA0)
- net UART4_RX: now reaches U1.15 (PA1)
- net SPI1_NSS: now reaches U1.20 (PA4)
- net SPI1_SCK: now reaches U1.21 (PA5)
- net SPI1_MISO: now reaches U1.22 (PA6)
- net SPI1_MOSI: now reaches U1.23 (PA7)
- net UART4_CTS: now reaches U1.26 (PB0)
- net at U1.30 (VCAP_1): now also C4.1
- net JTMS-SWDIO: now reaches U1.46 (PA13)
- net JTCK-SWCLK: now reaches U1.49 (PA14)
- net UART4_RTS: now reaches U1.50 (PA15)
- net I2C1_SCL: now reaches U1.58 (PB6)
- net I2C1_SCL: now also J3.4 (Pin_4)
- net I2C1_SDA: now reaches U1.59 (PB7)
- new net I2C1-SCL: R5.2
- new net I2C1-SDA: R6.2
Other:
- note added: "RTCCOnnector"
- note added: "crystal"
- moved on the sheet: C1, C2, C3, D1, J1, R1, R2, R3, R4, SW1, TP1, U2

Commit message: complete usb part ,reset part , SWD part
Parts:
- removed R3: R, Resistor_SMD:R_0805_2012Metric, symbol Device:R
- added C15, C16: 100n, symbol Device:C
- added J4: SWD, symbol Connector:Conn_01x05_Pin
- added R7: 10K, symbol Device:R
- added U4: CH340C, Package_SO:SOIC-16_3.9x9.9mm_P1.27mm, symbol Interface_USB:CH340C
- C3: value C -> 100n
- R4: value R -> 10K
Connections:
- net +3.3V is gone; now on net +3V3: R4.1
- net +3V3: now also C15.1, C16.1, J4.1 (Pin_1), U4.16 (VCC), U4.4 (V3)
- net +5V: now also U2.5 (VBUS)
- net GND: now also U2.2 (GND), C15.2, C16.2, J4.3 (Pin_3), R7.2, U4.1 (GND), U4.15 (R232)
- net JTCK-SWCLK: now also J4.4 (Pin_4)
- net JTMS-SWDIO: now also J4.2 (Pin_2)
- net RESET_STM_N: now also SW1.2, J4.5 (Pin_5)
- net UART4_RX: now also U4.2 (TXD)
- net UART4_TX: now also U4.3 (RXD)
- net USB_D+: now also U2.1 (I/O1)
- net USB_D-: now also U2.3 (I/O2)
- net CH340C UD-: now reaches U2.4 (I/O2)
- net CH340C UD-: now also U4.6 (UD-)
- net CH340C UD+: now reaches U2.6 (I/O1)
- net CH340C UD+: now also U4.5 (UD+)
- net at U1.60 (BOOT0): now also R7.1
- no-connect marks 0 -> 6
Other:
- note added: "静电保护装置"
- moved on the sheet: C13, C14, C3, J2, J3, R4, SW1, U2, U3

Commit message: complete .sch : add led*2 , mram , protection , transfer . wait for pcb part
Parts:
- removed C1: C, Capacitor_SMD:C_0805_2012Metric, symbol Device:C
- removed J1: Conn_01x05_Socket, Connector_PinHeader_2.54mm:PinHeader_1x05_P2.54mm_Vertical, symbol Connector:Conn_01x05_Socket
- removed TP1: TestPoint, TestPoint:TestPoint_Pad_D2.0mm, symbol Connector:TestPoint
- added D2: LED, LED_SMD:LED_Cree-XHP50_3V_HighDensity, symbol Device:LED
- added Q1, Q2: BSS138, Package_TO_SOT_SMD:SOT-23, symbol Transistor_FET:BSS138
- added R10, R11: 4.7K, Resistor_SMD:R_0805_2012Metric, symbol Device:R
- added R3: 10K, Resistor_SMD:R_0805_2012Metric, symbol Device:R
- added R4: 1K, Resistor_SMD:R_0805_2012Metric, symbol Device:R
- added R6: 10k, Resistor_SMD:R_0805_2012Metric, symbol Device:R
- added U1: PM004MNIATR, easyeda2kicad:SOP-8_L4.9-W3.9-P1.27-LS6.0-BL, symbol easyeda2kicad:PM004MNIATR
- C10: renamed from C11; footprint (none) -> Capacitor_SMD:C_0805_2012Metric
- C11: renamed from C9; footprint (none) -> Capacitor_SMD:C_0805_2012Metric
- C12: renamed from C13; footprint Package_QFP:PQFP-160_28x28mm_P0.65mm -> Capacitor_SMD:C_0805_2012Metric
- C13: renamed from C14; footprint Package_QFP:PQFP-160_28x28mm_P0.65mm -> Capacitor_SMD:C_0805_2012Metric
- C14: renamed from C15; footprint (none) -> Capacitor_SMD:C_0805_2012Metric
- C15: renamed from C16; footprint (none) -> Capacitor_SMD:C_0805_2012Metric
- C2: value C -> 100n; footprint Capacitor_SMD:C_0603_1608Metric -> Capacitor_SMD:C_0805_2012Metric
- C5: renamed from C4; footprint (none) -> Capacitor_SMD:C_0805_2012Metric
- C8: renamed from C10; footprint (none) -> Capacitor_SMD:C_0805_2012Metric
- C9: renamed from C12; footprint (none) -> Capacitor_SMD:C_0805_2012Metric
- D1: value LED GREEN -> LED; footprint LED_SMD:LED_0805_2012Metric -> LED_SMD:LED_Cree-XHP50_3V_HighDensity
- J1: renamed from J4; footprint (none) -> Connector_PinHeader_2.54mm:PinHeader_1x05_P2.54mm_Vertical
- R1: value R -> 10k
- R2: value R -> 1K; footprint Resistor_SMD:R_0603_1608Metric -> Resistor_SMD:R_0805_2012Metric
- R7: footprint (none) -> Resistor_SMD:R_0805_2012Metric
- R8: renamed from R5; value R -> 4.7K
- R9: renamed from R6; value R -> 4.7K
- renumbered C3 to C1, C5 to C3, C6 to C4, C7 to C6, C8 to C7, R4 to R5, U1 to U2, U2 to U4, U4 to U5
Connections:
- net I2C1-SCL is gone; now on net I2C1_SCL: R8.2
- net I2C1-SDA is gone; now on net I2C1_SDA: R9.2
- net +3V3: now also C2.1, R2.2, Q1.1 (G), Q2.1 (G), R3.1, U1.8 (VCC)
- net +5V: now also J3.2 (Pin_2), R10.1, R11.1
- net GND: now also C2.2, D1.1 (K), J2.SH (Shield), R1.2, D2.1 (K), R6.1, U1.4 (VSS)
- net I2C1_SCL: now also Q1.2 (S); no longer J3.4 (Pin_4)
- net I2C1_SDA: now also Q2.2 (S)
- net SPI1_MISO: now also U1.2 (SO/SIO[1])
- net SPI1_MOSI: now also U1.5 (SI/SO[0])
- net SPI1_NSS: now also R3.2, U1.1 (~{CE})
- net SPI1_SCK: now also U1.6 (CLK)
- net UART4_CTS: now also U5.14 (~{RTS})
- net UART4_RTS: now also U5.9 (~{CTS})
- net RUN_LED: now reaches U2.8 (PC0)
- net RUN_LED: now also R4.2
- net at D1.2 (A): now also R2.1
- net at R1.1: now also U1.3 (SIO[2])
- net RTC_SDA_5V: now reaches J3.3 (Pin_3)
- net RTC_SDA_5V: now also Q2.3 (D), R11.2
- new net: D2.2 (A), R4.1
- new net: R6.2, U1.7 (SIO[3])
- new net RTC_SCL_5V: J3.4 (Pin_4), Q1.3 (D), R10.2
- no-connect marks 6 -> 43
Other:
- note added: "RTCConnector"
- note added: "charger led"
- note added: "run_led"
- note added: "usb <-> urat 模块"
- note added: "双向电平转换_SCL"
- note added: "双向电平转换_SDA"
- note removed: "Connecteurs"
- note removed: "Debug STM32"
- note removed: "Footprint 0603"
- note removed: "Footprint 0805"
- note removed: "Point de Test"
- note removed: "RTCCOnnector"
- note removed: "Symboles Alim"
- moved on the sheet: C1, C10, C11, C12, C13, C3, C4, C6, C7, C8, C9, J1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

Commit message: start pcb design
Parts:
- D1, D2: footprint LED_SMD:LED_Cree-XHP50_3V_HighDensity -> LED_SMD:LED_0805_2012Metric
Changed lines of the file:
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@@
 			)
 		)
-		(property "Footprint" "LED_SMD:LED_Cree-XHP50_3V_HighDensity"
+		(property "Footprint" "LED_SMD:LED_0805_2012Metric"
 			(at 53.34 181.61 0)
 			(hide yes)
@@
 			)
 		)
-		(property "Footprint" "LED_SMD:LED_Cree-XHP50_3V_HighDensity"
+		(property "Footprint" "LED_SMD:LED_0805_2012Metric"
 			(at 52.07 162.56 0)
 			(hide yes)

Commit message: first version of PCB, a little change of shema
Parts:
- added J4: Conn_01x03_Socket, Connector_PinSocket_2.54mm:PinSocket_1x03_P2.54mm_Vertical, symbol Connector:Conn_01x03_Socket
Connections:
- net GND: now also J4.3 (Pin_3)
- net UART4_RX: now also J4.1 (Pin_1)
- net UART4_TX: now also J4.2 (Pin_2)
Changed lines of the file:
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@@
 	(text "静电保护装置"
 		(exclude_from_sim no)
-		(at 259.588 77.724 0)
+		(at 237.49 81.026 0)
 		(effects
 			(font
@@
 	(text "Protections"
 		(exclude_from_sim no)
-		(at 271.018 77.724 0)
+		(at 239.522 83.566 0)
 		(effects
 			(font
@@
 	(wire
 		(pts
+			(xy 257.81 72.39) (xy 269.24 72.39)
+		)
+		(stroke
+			(width 0)
+			(type default)
+		)
+	)
+	(wire
+		(pts
 			(xy 262.89 55.88) (xy 273.05 55.88)
 		)
@@
 	(wire
 		(pts
+			(xy 265.43 74.93) (xy 269.24 74.93)
+		)
+		(stroke
+			(width 0)
+			(type default)
+		)
+	)
+	(wire
+		(pts
 			(xy 158.75 97.79) (xy 170.18 97.79)
 		)
@@
 	(wire
 		(pts
-			(xy 33.02 86.36) (xy 45.72 86.36)
+			(xy 33.02 86.36) (xy 48.26 86.36)
 		)
 		(stroke
@@
 	(wire
 		(pts
+			(xy 257.81 69.85) (xy 269.24 69.85)
+		)
+		(stroke
+			(width 0)
+			(type default)
+		)
+	)
+	(wire
+		(pts
 			(xy 262.89 35.56) (xy 274.32 35.56)
 		)
@@
 	)
 	(label "JTCK-SWCLK"
-		(at 35.56 86.36 0)
+		(at 48.26 86.36 180)
 		(effects
 			(font
 				(size 1.27 1.27)
 			)
-			(justify left bottom)
+			(justify right bottom)
 		)
 	)
@@
 	)
 	(label "RESET_STM_N"
-		(at 35.56 88.9 0)
+		(at 48.26 88.9 180)
 		(effects
 			(font
 				(size 1.27 1.27)
 			)
-			(justify left bottom)
+			(justify right bottom)
 		)
 	)
@@
 		)
 	)
+	(label "UART4_RX"
+		(at 257.81 69.85 0)
+		(effects
+			(font
+				(size 1.27 1.27)
+			)
+			(justify left bottom)
+		)
+	)
 	(label "SPI1_NSS"
 		(at 27.94 142.24 0)
@@
 		)
 	)
-	(label "JTMS-SWDIO"
-		(at 36.83 81.28 0)
+	(label "UART4_TX"
+		(at 257.81 72.39 0)
 		(effects
 			(font
@@
 		)
 	)
+	(label "JTMS-SWDIO"
+		(at 49.53 81.28 180)
+		(effects
+			(font
+				(size 1.27 1.27)
+			)
+			(justify right bottom)
+		)
+	)
 	(label "RTC_SCL_5V"
 		(at 257.81 133.35 0)
@@
 	)
 	(symbol
+		(lib_id "Connector:Conn_01x03_Socket")
+		(at 274.32 72.39 0)
+		(unit 1)
+		(body_style 1)
+		(exclude_from_sim no)
+		(in_bom yes)
+		(on_board yes)
+		(in_pos_files yes)
+		(dnp no)
+		(fields_autoplaced yes)
+		(property "Reference" "J4"
+			(at 275.59 71.1199 0)
+			(show_name no)
+			(do_not_autoplace no)
+			(effects
+				(font
+					(size 1.27 1.27)
+				)
+				(justify left)
+			)
+		)
+		(property "Value" "Conn_01x03_Socket"
+			(at 275.59 73.6599 0)
+			(show_name no)
+			(do_not_autoplace no)
+			(effects
+				(font
+					(size 1.27 1.27)
+				)
+				(justify left)
+			)
+		)
+		(property "Footprint" "Connector_PinSocket_2.54mm:PinSocket_1x03_P2.54mm_Vertical"
+			(at 274.32 72.39 0)
+			(hide yes)
+			(show_name no)
+			(do_not_autoplace no)
+			(effects
+				(font
+					(size 1.27 1.27)
+				)
+			)
+		)
+		(property "Datasheet" ""
+			(at 274.32 72.39 0)
+			(hide yes)
+			(show_name no)
+			(do_not_autoplace no)
+			(effects
+				(font
+					(size 1.27 1.27)
+				)
+			)
+		)
+		(property "Description" "Generic connector, single row, 01x03, script generated"
+			(at 274.32 72.39 0)
+			(hide yes)
+			(show_name no)
+			(do_not_autoplace no)
+			(effects
+				(font
+					(size 1.27 1.27)
+				)
+			)
+		)
+		(pin "2"
+		)
+		(pin "1"
+		)
+		(pin "3"
+		)
+		(instances
+			(project "Projet_PCBPolytech_git"
+				(path "/4cd5a3a6-441a-4d49-b89e-ac57047910ed"
+					(reference "J4")
+					(unit 1)
+				)
+			)
+		)
+	)
+	(symbol
 		(lib_id "Device:C")
 		(at 120.65 36.83 0)
@@
 					(unit 1)
 				)
+			)
+		)
+	)
+	(symbol
+		(lib_id "power:GND")
+		(at 265.43 74.93 0)
+		(unit 1)
+		(body_style 1)
+		(exclude_from_sim no)
+		(in_bom yes)
+		(on_board yes)
+		(in_pos_files yes)
+		(dnp no)
+		(fields_autoplaced yes)
+		(property "Reference" "#PWR053"
+			(at 265.43 81.28 0)
+			(hide yes)
+			(show_name no)
+			(do_not_autoplace no)
+			(effects
+				(font
+					(size 1.27 1.27)
+				)
+			)
+		)
+		(property "Value" "GND"
+			(at 265.43 80.01 0)
+			(show_name no)
+			(do_not_autoplace no)
+			(effects
+				(font
+					(size 1.27 1.27)
+				)
+			)
+		)
+		(property "Footprint" ""
+			(at 265.43 74.93 0)
+			(hide yes)
+			(show_name no)
+			(do_not_autoplace no)
+			(effects
+				(font
+					(size 1.27 1.27)
+				)
+			)
+		)
+		(property "Datasheet" ""
+			(at 265.43 74.93 0)
+			(hide yes)
+			(show_name no)
+			(do_not_autoplace no)
+			(effects
+				(font
+					(size 1.27 1.27)
+				)
+			)
+		)
+		(property "Description" "Power symbol creates a global label with name \"GND\" , ground"
+			(at 265.43 74.93 0)
+			(hide yes)
+			(show_name no)
+			(do_not_autoplace no)
+			(effects
+				(font
+					(size 1.27 1.27)
+				)
+			)
+		)
+		(pin "1"
+		)
+		(instances
+			(project "Projet_PCBPolytech_git"
+				(path "/4cd5a3a6-441a-4d49-b89e-ac57047910ed"
+					(reference "#PWR053")
+					(unit 1)
+				)

Commit message: second version of PCB, connection
Other:
- note added: "VBAT"
- note added: "VDD"
- note added: "VDDA"
- note added: "boutton poussoir"
- note removed: "Exemple boutton poussoir"
- note removed: "Modèle à choisir + Footprint"
- moved on the sheet: C1, C12, C13, C2, C3, C4, C6, C7, J3, J4, R1, R3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
